File: Gigabit Ethernet.kicad_sch (KiCad schematic)
At the start: 29 parts, among them J6 RJ45_RB1-125B8G1A, J79 GLPLX-SMT-188S7-QQ-Y_G, U6 RTL8111H-CG-RH, U7 ULC0524P, U8 ULC0524P, Y1 25MHz

Commit message: hierarchical schema rework
Connections:
- net GbE_PCIe_CLK+ renamed GBE.CK+
- net GbE_PCIe_CLK- renamed GBE.CK-
- net GbE_PCIe_RX+ renamed GBE.RX+
- net GbE_PCIe_RX- renamed GBE.RX-
- net GbE_PCIe_TX+ renamed GBE.TX+
- net GbE_PCIe_TX- renamed GBE.TX-
Other:
- moved on the sheet: C33, C34, C35, C36, C37, C38, C39, C40, C41, C42, C43, C44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

Commit message: prod files created
Parts:
- removed C48: 100nF/50V, A_HDJ_Library:C_0402_1005Metric, symbol Device:C
- removed J6: RJ45_RB1-125B8G1A, A_HDJ_Library:RJ45_UDE_RB1-125B8G1A, symbol Connector:RJ45_RB1-125B8G1A
- added C151: 100nF/50V, Capacitor_SMD:C_0402_1005Metric, symbol Device:C_Small
- added R157: 1M/1%, A_HDJ_Library:R_0402_1005Metric, symbol Device:R_Small
- U81: renamed from U7; now fitted; now in the parts list
- U82: renamed from U8; now fitted; now in the parts list
- renumbered C36 to C100, C40 to C101, C44 to C102, C38 to C103, C42 to C104, C39 to C105, C46 to C106, C43 to C107, C47 to C108, C37 to C93, C41 to C94, C45 to C95, C89 to C96, C33 to C97, C34 to C98, C35 to C99, J79 to J80, R20 to R107, R21 to R108, R24 to R109, R25 to R110, R22 to R111, R23 to R112, U6 to U83, Y1 to Y78
Connections:
- net GND: now also C151.2, R157.2
- net LED1_1000: now also J80.11 (K_GREEN)
- net LED2_ACT: now also J80.13 (K_YELLOW)
- net at R110.1: now also J80.14 (A_YELLOW)
- net at R109.1: now also J80.12 (A_GREEN)
- net at J80.15 (MP1): now also J80.16 (MP2), C151.1, R157.1
Other:
- note added: "[GBE]"
- moved on the sheet: C96, J80, R109, R110
