File: Gigabit Ethernet.kicad_sch (KiCad schematic)
At the start: 29 parts, among them J80 GLPLX-SMT-188S7-QQ-Y_G, U81 ULC0524P, U82 ULC0524P, U83 RTL8111H-CG-RH, Y78 25MHz

Commit message: fix
Parts:
- R111: footprint A_HDJ_Library:R_0603_1608Metric -> A_HDJ_Library:R_0402_1005Metric
Changed lines of the file:
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@@
 			)
 		)
-		(property "Footprint" "A_HDJ_Library:R_0603_1608Metric"
+		(property "Footprint" "A_HDJ_Library:R_0402_1005Metric"
 			(at 106.68 119.888 90)
 			(effects
