File: M.2 E&M Key.kicad_sch (KiCad schematic)
At the start: 27 parts, among them J15 Bus_M.2_Socket_M, J16 Bus_M.2_Socket_E, U78 SMTWEM220STR, U79 SMTWEM220STR, U80 SMTWEM220STR

Commit message: hierarchical schema rework
Parts:
- C49, C50, C55, C56: value 220nF/50V -> 220n
- R34, R35: value 10K/1% -> 10K
Connections:
- net CON_PCIE_TX_1+ is gone; now on net TX+: C49.2, J15.49 (PETp0/SATA-A+)
- net CON_PCIE_TX_1- is gone; now on net TX-: C50.2, J15.47 (PETn0/SATA-A-)
- net CON_PCIE_TX_0+ renamed TX+
- net CON_PCIE_TX_0- renamed TX-
- net PCIE_RX_0+ renamed PCIE_E.RX+
- net PCIE_RX_0- renamed PCIE_E.RX-
- net PCIE_RX_1+ renamed PCIE_M.RX+
- net PCIE_RX_1- renamed PCIE_M.RX-
- net PCIE_TX_0+ renamed PCIE_E.TX+
- net PCIE_TX_0- renamed PCIE_E.TX-
- net PCIE_TX_1+ renamed PCIE_M.TX+
- net PCIE_TX_1- renamed PCIE_M.TX-
- net REFCLKE+ renamed PCIE_E.CKE+
- net REFCLKE- renamed PCIE_E.CKE-
- net REFCLKM+ renamed PCIE_M.CKE+
- net REFCLKM- renamed PCIE_M.CKE-
- net USB_2_P7+ renamed PCIE_E.P+
- net USB_2_P7- renamed PCIE_E.P-
Other:
- moved on the sheet: C49, C50, C51, C52, C53, C54, C55, C56, C57, C58, C59, C60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

Commit message: save
Connections:
- net TX+ renamed E_TX+
- net E_TX+: no longer C49.2, J15.49 (PETp0/SATA-A+)
- net TX- renamed E_TX-
- net E_TX-: no longer C50.2, J15.47 (PETn0/SATA-A-)
- new net M_TX+: C49.2, J15.49 (PETp0/SATA-A+)
- new net M_TX-: C50.2, J15.47 (PETn0/SATA-A-)
Changed lines of the file:
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@@
 		)
 	)
-	(label "TX-"
-		(at 201.93 71.12 0)
+	(label "E_TX-"
+		(at 200.66 71.12 0)
 		(effects
 			(font
@@
 		)
 	)
-	(label "TX+"
-		(at 64.77 68.58 0)
+	(label "M_TX+"
+		(at 63.5 68.58 0)
 		(effects
 			(font
@@
 		)
 	)
-	(label "TX+"
-		(at 201.93 68.58 0)
+	(label "E_TX+"
+		(at 200.66 68.58 0)
 		(effects
 			(font
@@
 		)
 	)
-	(label "TX-"
-		(at 64.77 71.12 0)
+	(label "M_TX-"
+		(at 63.5 71.12 0)
 		(effects
 			(font

Commit message: prod files created
Parts:
- TP79: renamed from TP2; now left out of the parts list
- renumbered C51 to C109, C57 to C110, C52 to C111, C58 to C112, C53 to C113, C59 to C114, C54 to C115, C60 to C116, C49 to C117, C55 to C118, C50 to C119, C56 to C120, D80 to D88, J15 to J83, J16 to J84, R32 to R113, R27 to R114, R34 to R115, R35 to R116, R30 to R117, R28 to R118, R29 to R119, R33 to R120, U78 to U84, U80 to U85, U79 to U86
Connections:
- net PCIE_E.CKE+ renamed PCIE_E.CK3+
- net PCIE_E.CKE- renamed PCIE_E.CK3-
- net PCIE_M.CKE+ renamed PCIE_M.CK0+
- net PCIE_M.CKE- renamed PCIE_M.CK0-
Other:
- note added: "[PCIE M.2]"
