File: PSU.kicad_sch (KiCad schematic)
At the start: 62 parts, among them Q8 2N7002, SW101 MK-11C04-G013, SW78 GT-TC193A-H0675-L1, U14 CH224K, U15 SY8253ADC, U16 SY8253ADC

Commit message: hierarchical schema rework
Other:
- moved on the sheet: C61, C64, C65, C67, C68, C70, C71, C72, C73, C74, C75, C76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

Commit message: prod files created
Parts:
- removed D18, D19, D20: SS54, A_HDJ_Library:D_SMA, symbol Device:D_Schottky
- added C128, C131: 100nF/50V, A_HDJ_Library:C_0402_1005Metric, symbol Device:C
- added Q82: AGM403A1, EasyEDA:DFN-8_L5.8-W4.9-P1.27-LS6.0-BL-1, symbol EasyEDA:AGM403A1
- added U88: LM74700, Package_TO_SOT_SMD:SOT-23-6, symbol Power_Management:LM74700
- renumbered C70 to C121, C72 to C122, C74 to C123, C76 to C124, C78 to C125, C80 to C126, C82 to C127, C64 to C129, C67 to C130, C65 to C132, C68 to C133, C71 to C134, C73 to C135, C75 to C136, C77 to C137, C79 to C138, C81 to C139, C83 to C140, C61 to C141, C91 to C142, C92 to C143, D24 to D89, D702 to D90, D12 to D91, D13 to D92, D14 to D93, D10 to D94, D11 to D95, D78 to D96, D79 to D97, L1 to L78, L2 to L79, Q8 to Q83, R53 to R121, R57 to R122, R58 to R123, R59 to R124, R46 to R125, R51 to R126, R60 to R127, R52 to R128, R36 to R129, R37 to R130, R43 to R131, R47 to R132, R49 to R133, R80 to R134, R81 to R135, SW101 to SW78, SW78 to SW79, TP13 to TP80, TP3 to TP81, TP10 to TP82, TP5 to TP83, TP6 to TP84, U15 to U87, U16 to U89, U14 to U90, USB80 to USB81
Connections:
- net +15V: now also C128.1, C131.1, Q82.1 (S), Q82.2 (S), Q82.3 (S), U88.3 (EN), U88.6 (ANODE)
- net GND: now also C128.2, U88.2 (GND)
- net VDC: now also Q82.5 (D), Q82.6 (D), Q82.7 (D), Q82.8 (D), Q82.9 (D), U88.4 (CATHODE)
- net SW1: now reaches C134.1, L79.1, U89.6 (SW)
- net SW2: now reaches C121.1, L78.1, U87.6 (SW)
- new net: C131.2, U88.1 (VCAP)
- new net: Q82.4 (G), U88.5 (GATE)
Other:
- note added: "[PSU]"
- moved on the sheet: TP81, TP82
