File: SENSORS.kicad_sch (KiCad schematic)
At the start: 4 parts, among them U33 SHT4x, U34 STCC4

Commit message: prod files created
Parts:
- renumbered C145 to C147, U34 to U92, U33 to U93
Other:
- note added: "[SENSORS]"
- moved on the sheet: C146, C147, U92, U93
