File: fan_temp.kicad_sch (KiCad schematic)
At the start: 24 parts, among them M1 Fan_4pin, M2 Fan_4pin, U81 B4B-PH-SM4-TBT(LF)(SN)

Commit message: prod files created
Parts:
- removed C85: 100nF/50V, Capacitor_SMD:C_0402_1005Metric, symbol Device:C
- added C145: 100nF/50V, Capacitor_SMD:C_0402_1005Metric, symbol Device:C
- renumbered C84 to C144, D26 to D98, D27 to D99, JP2 to JP78, M1 to M78, M2 to M79, R72 to R136, R64 to R137, R68 to R138, R69 to R139, R66 to R140, R73 to R143, R75 to R144, R74 to R147, R65 to R148, R70 to R149, R71 to R151, R67 to R152, R63 to R153, TH1 to TH78, TP11 to TP85, TP12 to TP86, U81 to U91
Connections:
- net GND: now also C145.2
- net at D99.1 (K), M79.2 (+), R143.1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: now also C145.1
- no-connect marks 0 -> 2
Other:
- note added: "[FAN]"
- moved on the sheet: C144, D98, D99, JP78, M78, M79, R136, R137, R138, R139, R140, R143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
